Commit message: Corrections to flamewheel model

File: rotors_description/urdf/flamewheel.xacro (robot description, xacro)
@@ -6,5 +6,5 @@
   <xacro:property name="use_mesh_file" value="true" />
   <xacro:property name="mesh_file" value="package://rotors_description/meshes/flamewheel.dae" />
-  <xacro:property name="mass" value="1.14" /> <!-- [kg] -->
+  <xacro:property name="mass" value="1.381" /> <!-- [kg] -->
   <xacro:property name="body_width" value="0.36" /> <!-- [m] -->
   <xacro:property name="body_height" value="0.1" /> <!-- [m] -->
@@ -23,4 +23,5 @@
   <xacro:property name="rotor_drag_coefficient" value="8.06428e-05" />
   <xacro:property name="rolling_moment_coefficient" value="0.000001" />
+  <xacro:property name="imu_z" value="0.04" />
   <!-- Property Blocks -->
   <xacro:property name="body_inertia">
@@ -44,4 +45,11 @@
     <xacro:insert_block name="body_inertia" />
   </xacro:multirotor_base_macro>
+  <!-- Link for IMU -->
+  <link name="${namespace}/imu_link" />
+  <joint name="${namespace}/base_to_imu_joint" type="fixed" >
+    <parent link="${namespace}/base_link" />
+    <child link="${namespace}/imu_link"/>
+    <origin xyz="0 0 ${imu_z}" rpy="0 0 0" />
+  </joint>
   <!-- Create macro for one arm with rotor -->
   <xacro:macro name="arm_with_rotor" params="num dir loc_is_front loc_is_right">
@@ -60,4 +68,10 @@
       <xacro:property name="loc_leftright" value="left" />
     </xacro:unless>
+    <link name="${namespace}/rotor_${num}_link" />
+    <joint name="${namespace}/base_to_rotor_${num}_joint" type="fixed" >
+      <parent link="${namespace}/base_link" />
+      <child link="${namespace}/rotor_${num}_link"/>
+      <origin xyz="${loc_is_front * arm_length / sqrt2} ${loc_is_right * arm_length / sqrt2} ${rotor_offset_top}" rpy="0 0 0" />
+    </joint>
     <xacro:vertical_rotor
       robot_namespace="${namespace}"
@@ -66,5 +80,5 @@
       motor_constant="${motor_constant}"
       moment_constant="${moment_constant}"
-      parent="${namespace}/base_link"
+      parent="${namespace}/rotor_${num}_link"
       mass_rotor="${mass_rotor}"
       radius_rotor="${radius_rotor}"
@@ -78,11 +92,12 @@
       use_own_mesh="false"
       mesh="">
-      <origin xyz="${loc_is_front * arm_length / sqrt2} ${loc_is_right * arm_length / sqrt2} ${rotor_offset_top}" rpy="0 0 0" />
+      <origin xyz="0 0 0" rpy="0 0 0" />
       <xacro:insert_block name="rotor_inertia" />
     </xacro:vertical_rotor>
   </xacro:macro>
-  <xacro:arm_with_rotor num="0" dir="ccw" loc_is_front="1" loc_is_right="1" />
-  <xacro:arm_with_rotor num="1" dir="ccw" loc_is_front="-1" loc_is_right="-1" />
-  <xacro:arm_with_rotor num="2" dir="cw" loc_is_front="1" loc_is_right="-1" />
-  <xacro:arm_with_rotor num="3" dir="cw" loc_is_front="-1" loc_is_right="1" />
+  <!-- Rotor config see https://docs.px4.io/master/en/airframes/airframe_reference.html#quadrotor-x -->
+  <xacro:arm_with_rotor num="1" dir="ccw" loc_is_front="1" loc_is_right="1" />
+  <xacro:arm_with_rotor num="2" dir="ccw" loc_is_front="-1" loc_is_right="-1" />
+  <xacro:arm_with_rotor num="3" dir="cw" loc_is_front="1" loc_is_right="-1" />
+  <xacro:arm_with_rotor num="4" dir="cw" loc_is_front="-1" loc_is_right="1" />
 </robot>

File: rotors_description/urdf/flamewheel_base.xacro (robot description, xacro)
@@ -11,5 +11,5 @@
   </xacro:if>
   <!-- Mount an ADIS16448 IMU. -->
-  <xacro:default_imu namespace="${namespace}" parent_link="${namespace}/base_link" />
+  <xacro:default_imu namespace="${namespace}" parent_link="${namespace}/imu_link" />
   <xacro:if value="$(arg enable_ground_truth)">
     <xacro:ground_truth_imu_and_odometry namespace="${namespace}" parent_link="${namespace}/base_link" />
